Commit message: Full mission in simulation: fake Xtion camera, cube detector, SO-100 IK and fake arm
- fake_robot.py: green cube on the Station 1 desk (random +-3 cm), blue place
  marker on Station 2, cube follows the jaws via TF gripper_tip; start_pose param
- fake_camera.py: renders the Xtion view (640x480) from TF camera_color_optical_frame
- cube_detector.py: HSV blob + ray / desk-plane intersection -> /detected/cube, /detected/station
- arm_control.py: SO-100 FK/IK from so_arm100.xml, pick/place/stow, small CLI
- fake_arm.py + robot_model.launch.py arm:=sim; URDF gets the camera mast and frames
- mission_nav2.py: real DETECT/PICK/PLACE (approach to 0.30 m, back off, fold);
  --nav-only keeps the driving-only practice
- mission.rviz, guide part 5, README run table; README junk line from PowerShell removed

Tested on Windows: Mission finished: succeeded in 207 s, cube placed 1.4 mm from the marker centre.

File: robot/kobuki_x2.urdf (robot description, URDF)
Before this commit: robot kobuki_x2, 13 links, 12 joints
Links:
- added link camera_color_optical_frame
- added link camera_link; visual box size=0.035 0.18 0.05
- added link camera_mast; visual cylinder length=0.24 radius=0.006
Joints:
- added joint camera_joint: type fixed, parent base_link, child camera_link, origin xyz=-0.04 0 0.42 rpy=0 0.61 0
- added joint camera_mast_joint: type fixed, parent base_link, child camera_mast, origin xyz=-0.055 0 0.2776 rpy=0 0 0
- added joint camera_optical_joint: type fixed, parent camera_link, child camera_color_optical_frame, origin xyz=0.02 0 0 rpy=-1.5708 0 -1.5708

Commit message: Demo-day step 3: real SO-100 driver, real camera tools, as-built robot
- Robot model rebuilt from the team's photos: two acrylic decks, battery,
  LiDAR front-right, SO-100 and Xtion working out of the rear; one link per
  colour so RViz shows the real colours. Positions marked MEASURE.
- Mission works out of the rear: park 0.65 m from the object, reverse to
  0.27 m, objects on the floor. A failed pick backs off to where the camera
  sees the object again.
- New: feetech.py, so100_driver.py, so100_calibrate.py (3 poses),
  camera_node.py (Xtion/OpenNI2 or webcam), hsv_tuner.py, camera_check.py.
- lidar_ros2.py drops returns within 0.24 m of the robot centre (battery and
  arm sit in the laser plane).
- docs/DEMO_DAY_TH.md: demo-day checklist with pictures; guides, README and
  handbook updated to the as-built layout.

Tested in the sim: full mission succeeded (229 s with the fake arm, 232 s
with so100_driver.py on virtual servos); camera_check found a planted
5/2 deg camera error and fixed it to 0.1 cm.

File: robot/kobuki_x2.urdf (robot description, URDF)
Before this commit: robot kobuki_x2, 16 links, 15 joints
Links:
- removed link camera_mast
- removed link lidar_deck
- added link battery; visual box size=0.045 0.003 0.045; visual box size=0.05 0.055 0.025
- added link battery_button; visual box size=0.004 0.03 0.03
- added link decks; visual mesh filename=MESH_URI/deck_plate.stl; visual mesh filename=MESH_URI/deck_plate.stl
- added link laser_cap; visual mesh filename=MESH_URI/ydlidar_x2_top.stl
- added link servo_terminal; visual box size=0.012 0.008 0.01
- added link standoffs; visual box size=0.10 0.06 0.02; visual cylinder length=0.06 radius=0.007
- added link white_plates; visual box size=0.09 0.075 0.005; visual box size=0.12 0.13 0.008
- link camera_link: geometry visual mesh filename=MESH_URI/xtion.stl
- link laser: geometry visual mesh filename=MESH_URI/ydlidar_x2_base.stl
Joints:
- removed joint camera_mast_joint
- removed joint lidar_deck_joint
- added joint battery_button_joint: type fixed, parent base_link, child battery_button, origin xyz=0 0 0 rpy=0 0 0
- added joint battery_joint: type fixed, parent base_link, child battery, origin xyz=0 0 0 rpy=0 0 0
- added joint decks_joint: type fixed, parent base_link, child decks, origin xyz=0 0 0 rpy=0 0 0
- added joint laser_cap_joint: type fixed, parent laser, child laser_cap, origin xyz=0 0 0 rpy=0 0 0
- added joint servo_terminal_joint: type fixed, parent base_link, child servo_terminal, origin xyz=0 0 0 rpy=0 0 0
- added joint standoffs_joint: type fixed, parent base_link, child standoffs, origin xyz=0 0 0 rpy=0 0 0
- added joint white_plates_joint: type fixed, parent base_link, child white_plates, origin xyz=0 0 0 rpy=0 0 0
- joint camera_joint: origin xyz=-0.04 0 0.42 rpy=0 0.61 0 -> xyz=-0.135 0 0.1775 rpy=0 0 3.14159
- joint camera_optical_joint: origin xyz=0.02 0 0 rpy=-1.5708 0 -1.5708 -> xyz=0.0175 0.045 0 rpy=-1.5708 0 -1.5708
- joint laser_joint: origin xyz=0 0 0.20 rpy=0 0 -1.5708 -> xyz=0.075 -0.035 0.247 rpy=0 0 -1.5708
- joint so100_mount_joint: origin xyz=0.06 0 0.1244 rpy=0 0 1.5708 -> xyz=-0.055 -0.03 0.208 rpy=0 0 -1.5708

Commit message: Final build: arm and Xtion work out of the front, TF from the 31 Oct photos
URDF (kobuki_x2.urdf, photo estimates marked MEASURE)
- so100_mount_joint -0.03 -0.02 0.208, yaw +90: the arm reaches out of the front
- camera_joint 0.14 0 0.1775, yaw 0: Xtion at the front edge of the bottom deck, looking forward
- laser_joint 0.085 0.085 0.247: LiDAR front left (yaw kept; re-run lidar_calib.py on the day)
- PINSEN battery standing behind the arm at the rear, DC-DC heatsink rear left, LiDAR USB box left
- MoveIt: rest/carry/home and all pick/place poses collision-free in the new layout;
  named pick/place poses recomputed for the cube 31 cm in front

Mission
- works forward on its own (WORK read from the arm mount): parks 0.65 m facing the object, drives in
- approach keeps the far view when the close look is more than 3 cm off: at 0.31 m the front camera
  cuts the cube off at the image bottom and the detector put it 4 cm too far
- Detect no longer resets the retry counter (a failing PICK looped forever)

Sim: the cube and the marker stand on 9 cm boxes as on demo day. Full mission with the front-facing
arm: succeeded in 215 s, cube grabbed 0.3 cm off-centre and released on the Station 2 marker.

Docs: REAL_DAY_TH.md for the front-facing build (+0.31, camera_check 0.65, pan direction check,
lidar_calib step), calibration texts say front/left, docs/UBUNTU_TH.md = plain Ubuntu 22.04 +
ROS 2 Humble from apt (no pixi), from git clone to the robot back home

File: robot/kobuki_x2.urdf (robot description, URDF)
Before this commit: robot kobuki_x2, 21 links, 20 joints
Links:
- link battery: geometry visual box size=0.003 0.045 0.045; visual box size=0.05 0.055 0.025
- link battery_button: geometry visual box size=0.03 0.004 0.03
- link servo_terminal: geometry visual box size=0.008 0.012 0.01
- link standoffs: geometry visual box size=0.09 0.07 0.03; visual cylinder length=0.06 radius=0.007
Joints:
- joint camera_joint: origin xyz=-0.135 0 0.1775 rpy=0 0 3.14159 -> xyz=0.14 0 0.1775 rpy=0 0 0
- joint laser_joint: origin xyz=0.075 -0.035 0.247 rpy=0 0 -1.5708 -> xyz=0.085 0.085 0.247 rpy=0 0 -1.5708
- joint so100_mount_joint: origin xyz=-0.055 -0.03 0.208 rpy=0 0 -1.5708 -> xyz=-0.03 -0.02 0.208 rpy=0 0 1.5708
